File: multi_expansion_board3/multi_expansion_board3.kicad_sch (KiCad schematic)
At the start: 46 parts, among them J1 Conn_01x20, J10 Conn_01x20, J11 Conn_01x20, J12 Conn_01x20, J13 Conn_01x20, J14 Conn_01x20, J15 Conn_01x20, J16 Conn_01x20, J17 Conn_01x20, J18 Conn_01x20, J19 Conn_01x04, J2 Conn_01x20, J20 Conn_01x04, J21 Conn_01x04, J22 Conn_01x04, J23 Conn_01x04, J24 Conn_01x04, J25 Conn_01x04, J26 Conn_01x02, J27 Barrel_Jack, J28 Screw_Terminal_01x02, J3 Conn_01x20, J4 Conn_01x20, J5 Conn_01x20, J6 Conn_01x20, J7 Conn_01x20, J8 Conn_01x20, J9 Conn_01x20, SW1 SW_Push, SW2 SW_Push, SW3 SW_Push, SW4 SW_SPST, U1 AMS1117-5.0

Commit message: A few tweaks to multi_expansion_board3.
Parts:
- added J1, J20: Conn_01x20, Custom:PinHeader_1x20_P2.54mm_Vertical_No_Silk, symbol Connector_Generic:Conn_01x20
- renumbered J9 to J10, J10 to J11, J11 to J12, J12 to J13, J13 to J14, J14 to J15, J15 to J16, J16 to J17, J17 to J18, J18 to J19, J1 to J2, J19 to J21, J20 to J22, J21 to J23, J22 to J24, J23 to J25, J24 to J26, J25 to J27, J2 to J3, J3 to J4, J4 to J5, J5 to J6, J6 to J7, J7 to J8, J8 to J9, J26 to PWR1, J27 to PWR2, J28 to PWR3
Connections:
- net Pin_1: now also J1.1 (Pin_1)
- net Pin_10: now also J1.10 (Pin_10)
- net Pin_11: now also J1.11 (Pin_11)
- net Pin_12: now also J1.12 (Pin_12)
- net Pin_13: now also J1.13 (Pin_13)
- net Pin_14: now also J1.14 (Pin_14)
- net Pin_15: now also J1.15 (Pin_15)
- net Pin_16: now also J1.16 (Pin_16)
- net Pin_17: now also J1.17 (Pin_17)
- net Pin_18: now also J1.18 (Pin_18)
- net Pin_19: now also J1.19 (Pin_19)
- net Pin_2: now also J1.2 (Pin_2)
- net Pin_20: now also J1.20 (Pin_20)
- net Pin_21: now also J20.20 (Pin_20)
- net Pin_22: now also J20.19 (Pin_19)
- net Pin_23: now also J20.18 (Pin_18)
- net Pin_24: now also J20.17 (Pin_17)
- net Pin_25: now also J20.16 (Pin_16)
- net Pin_26: now also J20.15 (Pin_15)
- net Pin_27: now also J20.14 (Pin_14)
- net Pin_28: now also J20.13 (Pin_13)
- net Pin_29: now also J20.12 (Pin_12)
- net Pin_3: now also J1.3 (Pin_3)
- net Pin_30: now also J20.11 (Pin_11)
- net Pin_31: now also J20.10 (Pin_10)
- net Pin_32: now also J20.9 (Pin_9)
- net Pin_33: now also J20.8 (Pin_8)
- net Pin_34: now also J20.7 (Pin_7)
- net Pin_35: now also J20.6 (Pin_6)
- net Pin_36: now also J20.5 (Pin_5)
- net Pin_37: now also J20.4 (Pin_4)
- net Pin_38: now also J20.3 (Pin_3)
- net Pin_39: now also J20.2 (Pin_2)
- net Pin_4: now also J1.4 (Pin_4)
- net Pin_40: now also J20.1 (Pin_1)
- net Pin_5: now also J1.5 (Pin_5)
- net Pin_6: now also J1.6 (Pin_6)
- net Pin_7: now also J1.7 (Pin_7)
- net Pin_8: now also J1.8 (Pin_8)
- net Pin_9: now also J1.9 (Pin_9)
Other:
- moved on the sheet: J21, J22, J23, J24, J25, J26, J27
