File: multi_expansion_board3/multi_expansion_board3_layout.kicad_pcb (KiCad board)
At the start: 2 copper layers, 91.4 x 96.5 mm, 500 parts, among them J1 Conn_01x20, J10 Conn_01x20, J11 Conn_01x20, J12 Conn_01x20, J13 Conn_01x20, J14 Conn_01x20, J15 Conn_01x20, J16 Conn_01x20, J17 Conn_01x20, J18 Conn_01x20, J19 Conn_01x04, J2 Conn_01x20, J20 Conn_01x04, J21 Conn_01x04, J22 Conn_01x04, J23 Conn_01x04, J24 Conn_01x04, J25 Conn_01x04, J26 Conn_01x02, J27 Barrel_Jack, J28 Screw_Terminal_01x02, J29 Conn_01x20, J3 Conn_01x20, J30 Conn_01x20, J31 Conn_01x20, J32 Conn_01x20, J33 Conn_01x20, J34 Conn_01x20, J35 Conn_01x20, J36 Conn_01x20, J37 Conn_01x20, J38 Conn_01x20, J39 Conn_01x20, J4 Conn_01x20, J40 Conn_01x20, J41 Conn_01x20, J42 Conn_01x20, J43 Conn_01x20, J44 Conn_01x20, J45 Conn_01x20, J46 Conn_01x20, J47 Conn_01x04, J48 Conn_01x04, J49 Conn_01x04, J5 Conn_01x20, J50 Conn_01x04, J51 Conn_01x04, J52 Conn_01x04, J53 Conn_01x04, J54 Conn_01x02, J55 Barrel_Jack, J56 Screw_Terminal_01x02, J6 Conn_01x20, J7 Conn_01x20, J8 Conn_01x20, J9 Conn_01x20, SW1 SW_Push, SW2 SW_Push, SW3 SW_Push, SW4 SW_SPST, SW5 SW_Push, SW6 SW_Push, SW7 SW_Push, SW8 SW_SPST, U1 AMS1117-5.0, U2 AMS1117-5.0

Commit message: A few tweaks to multi_expansion_board3.
Parts:
- removed J55: Barrel_Jack, Connector_BarrelJack:BarrelJack_Horizontal
- removed J56: Screw_Terminal_01x02, TerminalBlock:TerminalBlock_bornier-2_P5.08mm
- added J26: Conn_01x04, Custom:PinHeader_1x04_P2.54mm_Vertical_No_Silk, F.Cu at (48.3, 125.7)
- added J27: Conn_01x04, Custom:PinHeader_1x04_P2.54mm_Vertical_No_Silk, F.Cu at (48.3, 128.3)
- added J28: Conn_01x20, Custom:PinHeader_1x20_P2.54mm_Vertical_No_Silk, F.Cu at (91.4, 72.4)
- added PWR4: Conn_01x02, Connector_PinHeader_2.54mm:PinHeader_1x02_P2.54mm_Vertical, F.Cu at (120.7, 144.8)
- added PWR5: Barrel_Jack, Connector_BarrelJack:BarrelJack_Horizontal, F.Cu at (111.8, 144.8)
- added PWR6: Screw_Terminal_01x02, TerminalBlock:TerminalBlock_bornier-2_P5.08mm, F.Cu at (109.2, 153.7)
- J19, J20, J47: value Conn_01x04 -> Conn_01x20; footprint Custom:PinHeader_1x04_P2.54mm_Vertical_No_Silk -> Custom:PinHeader_1x20_P2.54mm_Vertical_No_Silk
- J54: value Conn_01x02 -> Conn_01x04; footprint Connector_PinHeader_2.54mm:PinHeader_1x02_P2.54mm_Vertical -> Custom:PinHeader_1x04_P2.54mm_Vertical_No_Silk
- moved J47 77.3 mm to (132.1, 72.4), turned to 0 degrees
- moved J19 76.7 mm to (85.1, 72.4), turned to 0 degrees
- moved J20 73.0 mm to (86.4, 72.4), turned to 0 degrees
- moved J54 31.4 mm to (94.0, 128.3)
- moved J10 17.8 mm to (57.1, 72.4)
- moved J24 11.4 mm to (48.3, 137.2)
- moved J23 10.2 mm to (48.3, 142.2)
- moved J49 7.62 mm to (94.0, 134.6)
- moved J52 6.35 mm to (94.0, 132.1)
- moved J50 5.08 mm to (94.0, 142.2)
- moved J48 5.08 mm to (94.0, 139.7)
- moved J51 5.08 mm to (94.0, 137.2)
- moved J25 3.81 mm to (48.3, 132.1)
- moved J21 2.54 mm to (48.3, 139.7)
- moved J53 2.54 mm to (94.0, 125.7)
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- renumbered J26 to PWR1, J27 to PWR2, J28 to PWR3
Connections:
- J10 pad 1: Pin_40 -> Pin_1
- J10 pad 10: Pin_31 -> Pin_10
- J10 pad 11: Pin_30 -> Pin_11
- J10 pad 12: Pin_29 -> Pin_12
- J10 pad 13: Pin_28 -> Pin_13
- J10 pad 14: Pin_27 -> Pin_14
- J10 pad 15: Pin_26 -> Pin_15
- J10 pad 16: Pin_25 -> Pin_16
- J10 pad 17: Pin_24 -> Pin_17
- J10 pad 18: Pin_23 -> Pin_18
- J10 pad 19: Pin_22 -> Pin_19
- J10 pad 2: Pin_39 -> Pin_2
- J10 pad 20: Pin_21 -> Pin_20
- J10 pad 3: Pin_38 -> Pin_3
- J10 pad 4: Pin_37 -> Pin_4
- J10 pad 5: Pin_36 -> Pin_5
- J10 pad 6: Pin_35 -> Pin_6
- J10 pad 7: Pin_34 -> Pin_7
- J10 pad 8: Pin_33 -> Pin_8
- J10 pad 9: Pin_32 -> Pin_9
- J19 pad 1: GND -> Pin_40
- J19 pad 2: GND -> Pin_39
- J19 pad 3: GND -> Pin_38
- J19 pad 4: GND -> Pin_37
- J20 pad 1: GND -> Pin_40
- J20 pad 2: GND -> Pin_39
- J20 pad 3: GND -> Pin_38
- J20 pad 4: GND -> Pin_37
- J21 pad 1: /VIN -> GND
- J21 pad 2: /VIN -> GND
- J21 pad 3: /VIN -> GND
- J21 pad 4: /VIN -> GND
- J22 pad 1: /+5V -> GND
- J22 pad 2: /+5V -> GND
- J22 pad 3: /+5V -> GND
- J22 pad 4: /+5V -> GND
- J23 pad 1: /+3V3 -> /VIN
- J23 pad 2: /+3V3 -> /VIN
- J23 pad 3: /+3V3 -> /VIN
- J23 pad 4: /+3V3 -> /VIN
- J24 pad 1: /SDA -> /+5V
- J24 pad 2: /SDA -> /+5V
- J24 pad 3: /SDA -> /+5V
- J24 pad 4: /SDA -> /+5V
- J25 pad 1: /SCL -> /+3V3
- J25 pad 2: /SCL -> /+3V3
- J25 pad 3: /SCL -> /+3V3
- J25 pad 4: /SCL -> /+3V3
- J47 pad 1: GND -> Pin_40
- J47 pad 2: GND -> Pin_39
- J47 pad 3: GND -> Pin_38
- J47 pad 4: GND -> Pin_37
- J49 pad 1: /VIN -> GND
- J49 pad 2: /VIN -> GND
- J49 pad 3: /VIN -> GND
- J49 pad 4: /VIN -> GND
- J50 pad 1: /+5V -> /VIN
- J50 pad 2: /+5V -> /VIN
- J50 pad 3: /+5V -> /VIN
- J50 pad 4: /+5V -> /VIN
- J51 pad 1: /+3V3 -> /+5V
- J51 pad 2: /+3V3 -> /+5V
- J51 pad 3: /+3V3 -> /+5V
- J51 pad 4: /+3V3 -> /+5V
- J52 pad 1: /SDA -> /+3V3
- J52 pad 2: /SDA -> /+3V3
- J52 pad 3: /SDA -> /+3V3
- J52 pad 4: /SDA -> /+3V3
- J53 pad 1: /SCL -> /SDA
- J53 pad 2: /SCL -> /SDA
- J53 pad 3: /SCL -> /SDA
- J53 pad 4: /SCL -> /SDA
- J54 pad 1: Net-(J26-Pin_1) -> /SCL
- J54 pad 2: GND -> /SCL
- PWR1 pad 1: Net-(J26-Pin_1) -> Net-(PWR1-Pin_1)
- PWR2 pad 1: Net-(J26-Pin_1) -> Net-(PWR1-Pin_1)
- PWR3 pad 1: Net-(J26-Pin_1) -> Net-(PWR1-Pin_1)
- SW4 pad 2: Net-(J26-Pin_1) -> Net-(PWR1-Pin_1)
- SW4 pad 5: Net-(J26-Pin_1) -> Net-(PWR1-Pin_1)
- SW8 pad 2: Net-(J26-Pin_1) -> Net-(PWR1-Pin_1)
- SW8 pad 5: Net-(J26-Pin_1) -> Net-(PWR1-Pin_1)
Routing:
- net Net-(PWR1-Pin_1): track 0.00 -> 80.0 mm
- net Net-(J26-Pin_1): track 80.0 -> 0.00 mm
