File: hub75_multi_mcu/hub75_multi_mcu.kicad_pcb (KiCad board)
At the start: 2 copper layers, 48.3 x 99.1 mm, 344 parts, among them J1 Conn_01x20, J10 Conn_01x20, J11 Conn_01x20, J12 Conn_01x20, J13 Conn_01x02, J14 Barrel_Jack, J15 Screw_Terminal_01x02, J16 Screw_Terminal_01x02, J17 Conn_02x08_Odd_Even, J2 Conn_01x20, J3 Conn_01x20, J4 Conn_01x20, J5 Conn_01x20, J6 Conn_01x20, J7 Conn_01x20, J8 Conn_01x20, J9 Conn_01x20, SW1 SW_SPST

Commit message: Add .gitignore.
Parts:
- removed J10, J11, J12, J9: Conn_01x20, Custom:PinHeader_1x20_P2.54mm_Vertical_No_Silk
- added C3: 0.1uF, Capacitor_SMD:C_0805_2012Metric_Pad1.18x1.45mm_HandSolder, B.Cu at (77.5, 93.3)
- added C4: 0.1uF, Capacitor_SMD:C_0805_2012Metric_Pad1.18x1.45mm_HandSolder, B.Cu at (77.5, 56.5)
- added JP322: SolderJumper_2_Open, Custom:SolderJumper-mini-2, B.Cu at (85.1, 57.8)
- added JP323: SolderJumper_2_Open, Custom:SolderJumper-mini-2, B.Cu at (85.1, 55.2)
- added JP324: SolderJumper_2_Open, Custom:SolderJumper-mini-2, B.Cu at (83.2, 57.8)
- added JP325: SolderJumper_2_Open, Custom:SolderJumper-mini-2, B.Cu at (83.2, 55.2)
- added JP326: SolderJumper_2_Open, Custom:SolderJumper-mini-2, B.Cu at (81.3, 57.8)
- added JP327: SolderJumper_2_Open, Custom:SolderJumper-mini-2, B.Cu at (81.3, 55.2)
- added JP328: SolderJumper_2_Open, Custom:SolderJumper-mini-2, B.Cu at (79.4, 57.8)
- added JP329: SolderJumper_2_Open, Custom:SolderJumper-mini-2, B.Cu at (79.4, 55.2)
- added JP330: SolderJumper_2_Open, Custom:SolderJumper-mini-2, B.Cu at (79.4, 92.1)
- added JP331: SolderJumper_2_Open, Custom:SolderJumper-mini-2, B.Cu at (79.4, 94.6)
- added JP332: SolderJumper_2_Open, Custom:SolderJumper-mini-2, B.Cu at (81.3, 92.1)
- added JP333: SolderJumper_2_Open, Custom:SolderJumper-mini-2, B.Cu at (81.3, 94.6)
- added JP334: SolderJumper_2_Open, Custom:SolderJumper-mini-2, B.Cu at (83.2, 92.1)
- added JP335: SolderJumper_2_Open, Custom:SolderJumper-mini-2, B.Cu at (83.2, 94.6)
- added JP336: SolderJumper_2_Open, Custom:SolderJumper-mini-2, B.Cu at (85.1, 92.1)
- added JP337: SolderJumper_2_Open, Custom:SolderJumper-mini-2, B.Cu at (85.1, 94.6)
- added U1: 74AHCT245, Package_SO:SSOP-20_5.3x7.2mm_P0.65mm, F.Cu at (81.3, 53.3)
- added U2: 74AHCT245, Package_SO:SSOP-20_5.3x7.2mm_P0.65mm, F.Cu at (81.3, 96.5)
- JP1: footprint Jumper:SolderJumper-2_P1.3mm_Open_RoundedPad1.0x1.5mm -> Custom:SolderJumper-mini-2
- SW1: value SW_SPST -> SW_DPDT; footprint Button_Switch_THT:SW_E-Switch_EG1271_SPDT -> Button_Switch_THT:SW_CuK_JS202011CQN_DPDT_Straight
- moved J15 28.1 mm to (102.9, 120.7), turned to 0 degrees
- moved J6 25.5 mm to (116.8, 50.8)
- moved J5 24.5 mm to (114.3, 50.8)
- moved J14 22.6 mm to (91.8, 113.8), turned to 90 degrees
- moved JP203 20.7 mm to (88.3, 53.3)
- moved JP204 20.7 mm to (88.3, 55.9)
- moved JP205 20.7 mm to (88.3, 58.4)
- moved JP206 20.7 mm to (88.3, 61.0)
- moved JP208 20.7 mm to (88.3, 66.0)
- moved JP210 20.7 mm to (88.3, 71.1)
- moved JP212 20.7 mm to (88.3, 76.2)
- moved JP214 20.7 mm to (88.3, 81.3)
- moved JP216 20.7 mm to (88.3, 86.4)
- moved JP217 20.7 mm to (88.3, 88.9)
- moved JP218 20.7 mm to (88.3, 91.4)
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Connections:
- D1 pad 1: Net-(D1-K) -> VCC
- J13 pad 1: Net-(J13-Pin_1) -> /VIN
- J13 pad 2: Net-(D1-K) -> GND
- J14 pad 1: Net-(J13-Pin_1) -> /VIN
- J14 pad 2: Net-(D1-K) -> GND
- J14 pad 3: Net-(D1-K) -> unconnected-(J14-Pad3)
- J15 pad 1: Net-(J13-Pin_1) -> /VIN
- J15 pad 2: Net-(D1-K) -> GND
- J16 pad 1: Net-(J13-Pin_1) -> /VIN
- J16 pad 2: Net-(D1-K) -> GND
- J17 pad 1: /IDC01 (R1) -> /IDC01
- J17 pad 10: /IDC10 (B) -> /IDC10
- J17 pad 11: /IDC11 (C) -> /IDC11
- J17 pad 12: /IDC12 (D) -> /IDC12
- J17 pad 13: /IDC13 (CLK) -> /IDC13
- J17 pad 14: /IDC14 (LAT) -> /IDC14
- J17 pad 15: /IDC15 (OE) -> /IDC15
- J17 pad 2: /IDC02 (G1) -> /IDC02
- J17 pad 3: /IDC03 (B1) -> /IDC03
- J17 pad 5: /IDC05 (R2) -> /IDC05
- J17 pad 6: /IDC06 (G2) -> /IDC06
- J17 pad 7: /IDC07 (B2) -> /IDC07
- J17 pad 8: /IDC08 (E) -> /IDC08
- J17 pad 9: /IDC09 (A) -> /IDC09
- J5 pad 1: Pin_1 -> Pin_40
- J5 pad 10: Pin_10 -> Pin_31
- J5 pad 11: Pin_11 -> Pin_30
- J5 pad 12: Pin_12 -> Pin_29
- J5 pad 13: Pin_13 -> Pin_28
- J5 pad 14: Pin_14 -> Pin_27
- J5 pad 15: Pin_15 -> Pin_26
- J5 pad 16: Pin_16 -> Pin_25
- J5 pad 17: Pin_17 -> Pin_24
- J5 pad 18: Pin_18 -> Pin_23
- J5 pad 19: Pin_19 -> Pin_22
- J5 pad 2: Pin_2 -> Pin_39
- J5 pad 20: Pin_20 -> Pin_21
- J5 pad 3: Pin_3 -> Pin_38
- J5 pad 4: Pin_4 -> Pin_37
- J5 pad 5: Pin_5 -> Pin_36
- J5 pad 6: Pin_6 -> Pin_35
- J5 pad 7: Pin_7 -> Pin_34
- J5 pad 8: Pin_8 -> Pin_33
- J5 pad 9: Pin_9 -> Pin_32
- J6 pad 1: Pin_1 -> Pin_40
- J6 pad 10: Pin_10 -> Pin_31
- J6 pad 11: Pin_11 -> Pin_30
- J6 pad 12: Pin_12 -> Pin_29
- J6 pad 13: Pin_13 -> Pin_28
- J6 pad 14: Pin_14 -> Pin_27
- J6 pad 15: Pin_15 -> Pin_26
- J6 pad 16: Pin_16 -> Pin_25
- J6 pad 17: Pin_17 -> Pin_24
- J6 pad 18: Pin_18 -> Pin_23
- J6 pad 19: Pin_19 -> Pin_22
- J6 pad 2: Pin_2 -> Pin_39
- J6 pad 20: Pin_20 -> Pin_21
- J6 pad 3: Pin_3 -> Pin_38
- J6 pad 4: Pin_4 -> Pin_37
- J6 pad 5: Pin_5 -> Pin_36
- J6 pad 6: Pin_6 -> Pin_35
- J6 pad 7: Pin_7 -> Pin_34
- J6 pad 8: Pin_8 -> Pin_33
- J6 pad 9: Pin_9 -> Pin_32
- JP1 pad 1: Net-(D1-K) -> GND
- JP1 pad 2: GND -> VCC
- JP100 pad 2: /IDC03 (B1) -> /B1
- JP101 pad 2: /IDC03 (B1) -> /B1
- JP102 pad 2: /IDC05 (R2) -> /R2
- JP103 pad 2: /IDC05 (R2) -> /R2
- JP104 pad 2: /IDC05 (R2) -> /R2
- JP105 pad 2: /IDC05 (R2) -> /R2
- JP106 pad 2: /IDC05 (R2) -> /R2
- JP107 pad 2: /IDC05 (R2) -> /R2
- JP108 pad 2: /IDC05 (R2) -> /R2
- JP109 pad 2: /IDC05 (R2) -> /R2
- JP110 pad 2: /IDC05 (R2) -> /R2
- JP111 pad 2: /IDC05 (R2) -> /R2
- JP112 pad 2: /IDC05 (R2) -> /R2
- JP113 pad 2: /IDC05 (R2) -> /R2
- JP114 pad 2: /IDC05 (R2) -> /R2
- JP115 pad 2: /IDC05 (R2) -> /R2
- JP116 pad 2: /IDC05 (R2) -> /R2
- JP117 pad 2: /IDC05 (R2) -> /R2
- JP118 pad 2: /IDC05 (R2) -> /R2
- JP119 pad 2: /IDC05 (R2) -> /R2
- JP120 pad 2: /IDC05 (R2) -> /R2
- JP121 pad 2: /IDC05 (R2) -> /R2
- JP122 pad 2: /IDC06 (G2) -> /G2
- JP123 pad 2: /IDC06 (G2) -> /G2
- JP124 pad 2: /IDC06 (G2) -> /G2
- JP125 pad 2: /IDC06 (G2) -> /G2
- JP126 pad 2: /IDC06 (G2) -> /G2
- JP127 pad 2: /IDC06 (G2) -> /G2
- JP128 pad 2: /IDC06 (G2) -> /G2
- JP129 pad 2: /IDC06 (G2) -> /G2
- JP130 pad 2: /IDC06 (G2) -> /G2
- JP131 pad 2: /IDC06 (G2) -> /G2
- JP132 pad 2: /IDC06 (G2) -> /G2
- JP133 pad 2: /IDC06 (G2) -> /G2
- JP134 pad 2: /IDC06 (G2) -> /G2
- JP135 pad 2: /IDC06 (G2) -> /G2
- JP136 pad 2: /IDC06 (G2) -> /G2
- JP137 pad 2: /IDC06 (G2) -> /G2
- JP138 pad 2: /IDC06 (G2) -> /G2
- JP139 pad 2: /IDC06 (G2) -> /G2
- JP140 pad 2: /IDC06 (G2) -> /G2
- JP141 pad 2: /IDC06 (G2) -> /G2
- JP142 pad 2: /IDC07 (B2) -> /B2
- JP143 pad 2: /IDC07 (B2) -> /B2
- JP144 pad 2: /IDC07 (B2) -> /B2
- JP145 pad 2: /IDC07 (B2) -> /B2
- JP146 pad 2: /IDC07 (B2) -> /B2
- JP147 pad 2: /IDC07 (B2) -> /B2
- JP148 pad 2: /IDC07 (B2) -> /B2
- JP149 pad 2: /IDC07 (B2) -> /B2
- JP150 pad 2: /IDC07 (B2) -> /B2
- JP151 pad 2: /IDC07 (B2) -> /B2
- JP152 pad 2: /IDC07 (B2) -> /B2
- JP153 pad 2: /IDC07 (B2) -> /B2
- JP154 pad 2: /IDC07 (B2) -> /B2
- JP155 pad 2: /IDC07 (B2) -> /B2
- JP156 pad 2: /IDC07 (B2) -> /B2
- JP157 pad 2: /IDC07 (B2) -> /B2
- JP158 pad 2: /IDC07 (B2) -> /B2
- JP159 pad 2: /IDC07 (B2) -> /B2
- JP160 pad 2: /IDC07 (B2) -> /B2
- JP161 pad 2: /IDC07 (B2) -> /B2
- JP162 pad 2: /IDC08 (E) -> /E
- JP163 pad 2: /IDC08 (E) -> /E
- JP164 pad 2: /IDC08 (E) -> /E
- JP165 pad 2: /IDC08 (E) -> /E
- JP166 pad 2: /IDC08 (E) -> /E
- JP167 pad 2: /IDC08 (E) -> /E
- JP168 pad 2: /IDC08 (E) -> /E
- JP169 pad 2: /IDC08 (E) -> /E
- JP170 pad 2: /IDC08 (E) -> /E
- JP171 pad 2: /IDC08 (E) -> /E
- JP172 pad 2: /IDC08 (E) -> /E
- JP173 pad 2: /IDC08 (E) -> /E
- JP174 pad 2: /IDC08 (E) -> /E
- JP175 pad 2: /IDC08 (E) -> /E
- JP176 pad 2: /IDC08 (E) -> /E
- JP177 pad 2: /IDC08 (E) -> /E
- JP178 pad 2: /IDC08 (E) -> /E
- JP179 pad 2: /IDC08 (E) -> /E
- JP180 pad 2: /IDC08 (E) -> /E
- JP181 pad 2: /IDC08 (E) -> /E
- JP182 pad 2: /IDC09 (A) -> /A
- JP183 pad 2: /IDC09 (A) -> /A
- JP184 pad 2: /IDC09 (A) -> /A
- JP185 pad 2: /IDC09 (A) -> /A
- JP186 pad 2: /IDC09 (A) -> /A
- JP187 pad 2: /IDC09 (A) -> /A
- JP188 pad 2: /IDC09 (A) -> /A
- JP189 pad 2: /IDC09 (A) -> /A
- JP190 pad 2: /IDC09 (A) -> /A
- JP191 pad 2: /IDC09 (A) -> /A
- JP192 pad 2: /IDC09 (A) -> /A
- JP193 pad 2: /IDC09 (A) -> /A
- JP194 pad 2: /IDC09 (A) -> /A
- JP195 pad 2: /IDC09 (A) -> /A
- JP196 pad 2: /IDC09 (A) -> /A
- JP197 pad 2: /IDC09 (A) -> /A
- JP198 pad 2: /IDC09 (A) -> /A
- JP199 pad 2: /IDC09 (A) -> /A
- JP200 pad 2: /IDC09 (A) -> /A
- JP201 pad 2: /IDC09 (A) -> /A
- JP202 pad 2: /IDC10 (B) -> /B
- JP203 pad 2: /IDC10 (B) -> /B
- JP204 pad 2: /IDC10 (B) -> /B
- JP205 pad 2: /IDC10 (B) -> /B
- JP206 pad 2: /IDC10 (B) -> /B
- JP207 pad 2: /IDC10 (B) -> /B
- JP208 pad 2: /IDC10 (B) -> /B
- JP209 pad 2: /IDC10 (B) -> /B
- JP210 pad 2: /IDC10 (B) -> /B
- JP211 pad 2: /IDC10 (B) -> /B
- JP212 pad 2: /IDC10 (B) -> /B
- JP213 pad 2: /IDC10 (B) -> /B
- JP214 pad 2: /IDC10 (B) -> /B
- JP215 pad 2: /IDC10 (B) -> /B
- JP216 pad 2: /IDC10 (B) -> /B
- JP217 pad 2: /IDC10 (B) -> /B
- JP218 pad 2: /IDC10 (B) -> /B
- JP219 pad 2: /IDC10 (B) -> /B
- JP220 pad 2: /IDC10 (B) -> /B
- JP221 pad 2: /IDC10 (B) -> /B
- JP222 pad 2: /IDC11 (C) -> /C
- JP223 pad 2: /IDC11 (C) -> /C
- JP224 pad 2: /IDC11 (C) -> /C
- JP225 pad 2: /IDC11 (C) -> /C
- JP226 pad 2: /IDC11 (C) -> /C
- JP227 pad 2: /IDC11 (C) -> /C
- JP228 pad 2: /IDC11 (C) -> /C
- JP229 pad 2: /IDC11 (C) -> /C
- JP230 pad 2: /IDC11 (C) -> /C
- JP231 pad 2: /IDC11 (C) -> /C
- JP232 pad 2: /IDC11 (C) -> /C
- JP233 pad 2: /IDC11 (C) -> /C
- JP234 pad 2: /IDC11 (C) -> /C
- JP235 pad 2: /IDC11 (C) -> /C
- JP236 pad 2: /IDC11 (C) -> /C
- JP237 pad 2: /IDC11 (C) -> /C
- JP238 pad 2: /IDC11 (C) -> /C
- JP239 pad 2: /IDC11 (C) -> /C
- JP240 pad 2: /IDC11 (C) -> /C
- JP241 pad 2: /IDC11 (C) -> /C
- JP242 pad 2: /IDC12 (D) -> /D
- JP243 pad 2: /IDC12 (D) -> /D
- JP244 pad 2: /IDC12 (D) -> /D
- JP245 pad 2: /IDC12 (D) -> /D
- JP246 pad 2: /IDC12 (D) -> /D
- JP247 pad 2: /IDC12 (D) -> /D
- JP248 pad 2: /IDC12 (D) -> /D
- JP249 pad 2: /IDC12 (D) -> /D
- JP250 pad 2: /IDC12 (D) -> /D
- JP251 pad 2: /IDC12 (D) -> /D
- JP252 pad 2: /IDC12 (D) -> /D
- JP253 pad 2: /IDC12 (D) -> /D
- JP254 pad 2: /IDC12 (D) -> /D
- JP255 pad 2: /IDC12 (D) -> /D
- JP256 pad 2: /IDC12 (D) -> /D
- JP257 pad 2: /IDC12 (D) -> /D
- JP258 pad 2: /IDC12 (D) -> /D
- JP259 pad 2: /IDC12 (D) -> /D
- JP260 pad 2: /IDC12 (D) -> /D
- JP261 pad 2: /IDC12 (D) -> /D
- JP262 pad 2: /IDC13 (CLK) -> /CLK
- JP263 pad 2: /IDC13 (CLK) -> /CLK
- JP264 pad 2: /IDC13 (CLK) -> /CLK
- JP265 pad 2: /IDC13 (CLK) -> /CLK
- JP266 pad 2: /IDC13 (CLK) -> /CLK
- JP267 pad 2: /IDC13 (CLK) -> /CLK
- JP268 pad 2: /IDC13 (CLK) -> /CLK
- JP269 pad 2: /IDC13 (CLK) -> /CLK
- JP270 pad 2: /IDC13 (CLK) -> /CLK
- JP271 pad 2: /IDC13 (CLK) -> /CLK
- JP272 pad 2: /IDC13 (CLK) -> /CLK
- JP273 pad 2: /IDC13 (CLK) -> /CLK
- JP274 pad 2: /IDC13 (CLK) -> /CLK
- JP275 pad 2: /IDC13 (CLK) -> /CLK
- JP276 pad 2: /IDC13 (CLK) -> /CLK
- JP277 pad 2: /IDC13 (CLK) -> /CLK
- JP278 pad 2: /IDC13 (CLK) -> /CLK
- JP279 pad 2: /IDC13 (CLK) -> /CLK
- JP280 pad 2: /IDC13 (CLK) -> /CLK
- JP281 pad 2: /IDC13 (CLK) -> /CLK
- JP282 pad 2: /IDC14 (LAT) -> /LAT
- JP283 pad 2: /IDC14 (LAT) -> /LAT
- JP284 pad 2: /IDC14 (LAT) -> /LAT
- JP285 pad 2: /IDC14 (LAT) -> /LAT
- JP286 pad 2: /IDC14 (LAT) -> /LAT
- JP287 pad 2: /IDC14 (LAT) -> /LAT
- JP288 pad 2: /IDC14 (LAT) -> /LAT
- JP289 pad 2: /IDC14 (LAT) -> /LAT
- JP290 pad 2: /IDC14 (LAT) -> /LAT
- JP291 pad 2: /IDC14 (LAT) -> /LAT
- JP292 pad 2: /IDC14 (LAT) -> /LAT
- JP293 pad 2: /IDC14 (LAT) -> /LAT
- JP294 pad 2: /IDC14 (LAT) -> /LAT
- JP295 pad 2: /IDC14 (LAT) -> /LAT
- JP296 pad 2: /IDC14 (LAT) -> /LAT
- JP297 pad 2: /IDC14 (LAT) -> /LAT
- JP298 pad 2: /IDC14 (LAT) -> /LAT
- JP299 pad 2: /IDC14 (LAT) -> /LAT
- JP300 pad 2: /IDC14 (LAT) -> /LAT
- JP301 pad 2: /IDC14 (LAT) -> /LAT
- JP302 pad 2: /IDC15 (OE) -> /OE
- JP303 pad 2: /IDC15 (OE) -> /OE
- JP304 pad 2: /IDC15 (OE) -> /OE
- JP305 pad 2: /IDC15 (OE) -> /OE
- JP306 pad 2: /IDC15 (OE) -> /OE
- JP307 pad 2: /IDC15 (OE) -> /OE
- JP308 pad 2: /IDC15 (OE) -> /OE
- JP309 pad 2: /IDC15 (OE) -> /OE
- JP310 pad 2: /IDC15 (OE) -> /OE
- JP311 pad 2: /IDC15 (OE) -> /OE
- JP312 pad 2: /IDC15 (OE) -> /OE
- JP313 pad 2: /IDC15 (OE) -> /OE
- JP314 pad 2: /IDC15 (OE) -> /OE
- JP315 pad 2: /IDC15 (OE) -> /OE
- JP316 pad 2: /IDC15 (OE) -> /OE
- JP317 pad 2: /IDC15 (OE) -> /OE
- JP318 pad 2: /IDC15 (OE) -> /OE
- JP319 pad 2: /IDC15 (OE) -> /OE
- JP320 pad 2: /IDC15 (OE) -> /OE
- JP321 pad 2: /IDC15 (OE) -> /OE
- JP42 pad 2: /IDC01 (R1) -> /R1
- JP43 pad 2: /IDC01 (R1) -> /R1
- JP44 pad 2: /IDC01 (R1) -> /R1
- JP45 pad 2: /IDC01 (R1) -> /R1
- JP46 pad 2: /IDC01 (R1) -> /R1
- JP47 pad 2: /IDC01 (R1) -> /R1
- JP48 pad 2: /IDC01 (R1) -> /R1
- JP49 pad 2: /IDC01 (R1) -> /R1
- JP50 pad 2: /IDC01 (R1) -> /R1
- JP51 pad 2: /IDC01 (R1) -> /R1
- JP52 pad 2: /IDC01 (R1) -> /R1
- JP53 pad 2: /IDC01 (R1) -> /R1
- JP54 pad 2: /IDC01 (R1) -> /R1
- JP55 pad 2: /IDC01 (R1) -> /R1
- JP56 pad 2: /IDC01 (R1) -> /R1
- JP57 pad 2: /IDC01 (R1) -> /R1
- JP58 pad 2: /IDC01 (R1) -> /R1
- JP59 pad 2: /IDC01 (R1) -> /R1
- JP60 pad 2: /IDC01 (R1) -> /R1
- JP61 pad 2: /IDC01 (R1) -> /R1
- JP62 pad 2: /IDC02 (G1) -> /G1
- JP63 pad 2: /IDC02 (G1) -> /G1
- JP64 pad 2: /IDC02 (G1) -> /G1
- JP65 pad 2: /IDC02 (G1) -> /G1
- JP66 pad 2: /IDC02 (G1) -> /G1
- JP67 pad 2: /IDC02 (G1) -> /G1
- JP68 pad 2: /IDC02 (G1) -> /G1
- JP69 pad 2: /IDC02 (G1) -> /G1
- JP70 pad 2: /IDC02 (G1) -> /G1
- JP71 pad 2: /IDC02 (G1) -> /G1
- JP72 pad 2: /IDC02 (G1) -> /G1
- JP73 pad 2: /IDC02 (G1) -> /G1
- JP74 pad 2: /IDC02 (G1) -> /G1
- JP75 pad 2: /IDC02 (G1) -> /G1
- JP76 pad 2: /IDC02 (G1) -> /G1
- JP77 pad 2: /IDC02 (G1) -> /G1
- JP78 pad 2: /IDC02 (G1) -> /G1
- JP79 pad 2: /IDC02 (G1) -> /G1
- JP80 pad 2: /IDC02 (G1) -> /G1
- JP81 pad 2: /IDC02 (G1) -> /G1
- JP82 pad 2: /IDC03 (B1) -> /B1
- JP83 pad 2: /IDC03 (B1) -> /B1
- JP84 pad 2: /IDC03 (B1) -> /B1
- JP85 pad 2: /IDC03 (B1) -> /B1
- JP86 pad 2: /IDC03 (B1) -> /B1
- JP87 pad 2: /IDC03 (B1) -> /B1
- JP88 pad 2: /IDC03 (B1) -> /B1
- JP89 pad 2: /IDC03 (B1) -> /B1
- JP90 pad 2: /IDC03 (B1) -> /B1
- JP91 pad 2: /IDC03 (B1) -> /B1
- JP92 pad 2: /IDC03 (B1) -> /B1
- JP93 pad 2: /IDC03 (B1) -> /B1
- JP94 pad 2: /IDC03 (B1) -> /B1
- JP95 pad 2: /IDC03 (B1) -> /B1
- JP96 pad 2: /IDC03 (B1) -> /B1
- JP97 pad 2: /IDC03 (B1) -> /B1
- JP98 pad 2: /IDC03 (B1) -> /B1
- JP99 pad 2: /IDC03 (B1) -> /B1
- SW1 pad 1: Net-(J13-Pin_1) -> unconnected-(SW1A-A-Pad1)
- SW1 pad 2: VCC -> /VIN
- SW1 pad 3: (no net) -> GND
- SW1 pad 4: (no net) -> unconnected-(SW1B-A-Pad4)
- SW1 pad 5: (no net) -> GND
- SW1 pad 6: (no net) -> GND
Routing:
- net /IDC01 (R1): track 113.0 -> 0.00 mm
- net /IDC05 (R2): track 112.3 -> 0.00 mm
- net /IDC03 (B1): track 112.2 -> 0.00 mm
- net /IDC07 (B2): track 110.7 -> 0.00 mm
- net /IDC02 (G1): track 109.7 -> 0.00 mm
- net /IDC06 (G2): track 108.6 -> 0.00 mm
- net /A: track 0.00 -> 95.2 mm, vias 0 -> 1
- net /B2: track 0.00 -> 91.6 mm, vias 0 -> 1
- net /R2: track 0.00 -> 90.2 mm, vias 0 -> 1
- net /IDC09 (A): track 89.5 -> 0.00 mm
- net /IDC10 (B): track 88.8 -> 0.00 mm
- net /C: track 0.00 -> 88.3 mm, vias 0 -> 1
- net /CLK: track 0.00 -> 87.3 mm, vias 0 -> 1
- net /B1: track 0.00 -> 83.5 mm, vias 0 -> 1
- net /R1: track 0.00 -> 82.4 mm, vias 0 -> 1
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Other:
- board text added: "left pins lower pads"
- board text added: "right pins upper pads"
- board text removed: "HUB75 MULTI MCU"
- board text removed: "Lower-left"
- board text removed: "Upper-right"
