File: hub75_multi_mcu/hub75_multi_mcu.kicad_sch (KiCad schematic)
At the start: 20 parts, among them J1 Conn_01x20, J10 Conn_01x20, J11 Conn_01x20, J12 Conn_01x20, J13 Conn_01x02, J14 Barrel_Jack, J15 Screw_Terminal_01x02, J16 Screw_Terminal_01x02, J17 Conn_02x08_Odd_Even, J2 Conn_01x20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

Commit message: Add .gitignore.
Parts:
- removed J10, J11, J12, J9: Conn_01x20, Custom:PinHeader_1x20_P2.54mm_Vertical_No_Silk, symbol Connector_Generic:Conn_01x20
- removed SW1: SW_SPST, Button_Switch_THT:SW_E-Switch_EG1271_SPDT, symbol Switch:SW_SPST
- added SW1: SW_DPDT, Button_Switch_THT:SW_CuK_JS202011CQN_DPDT_Straight, symbol Switch:SW_DPDT_x2
- JP1: footprint Jumper:SolderJumper-2_P1.3mm_Open_RoundedPad1.0x1.5mm -> Custom:SolderJumper-mini-2
Connections:
- net GND: now also J13.2 (Pin_2), J14.2, J15.2 (Pin_2), J16.2 (Pin_2), JP1.1 (A), SW1.3 (C), SW1.5 (B), SW1.6 (C); no longer JP1.2 (B)
- net Pin_1: no longer J5.1 (Pin_1), J6.1 (Pin_1)
- net Pin_10: no longer J5.10 (Pin_10), J6.10 (Pin_10)
- net Pin_11: no longer J5.11 (Pin_11), J6.11 (Pin_11)
- net Pin_12: no longer J5.12 (Pin_12), J6.12 (Pin_12)
- net Pin_13: no longer J5.13 (Pin_13), J6.13 (Pin_13)
- net Pin_14: no longer J5.14 (Pin_14), J6.14 (Pin_14)
- net Pin_15: no longer J5.15 (Pin_15), J6.15 (Pin_15)
- net Pin_16: no longer J5.16 (Pin_16), J6.16 (Pin_16)
- net Pin_17: no longer J5.17 (Pin_17), J6.17 (Pin_17)
- net Pin_18: no longer J5.18 (Pin_18), J6.18 (Pin_18)
- net Pin_19: no longer J5.19 (Pin_19), J6.19 (Pin_19)
- net Pin_2: no longer J5.2 (Pin_2), J6.2 (Pin_2)
- net Pin_20: no longer J5.20 (Pin_20), J6.20 (Pin_20)
- net Pin_21: now also J5.20 (Pin_20), J6.20 (Pin_20)
- net Pin_22: now also J5.19 (Pin_19), J6.19 (Pin_19)
- net Pin_23: now also J5.18 (Pin_18), J6.18 (Pin_18)
- net Pin_24: now also J5.17 (Pin_17), J6.17 (Pin_17)
- net Pin_25: now also J5.16 (Pin_16), J6.16 (Pin_16)
- net Pin_26: now also J5.15 (Pin_15), J6.15 (Pin_15)
- net Pin_27: now also J5.14 (Pin_14), J6.14 (Pin_14)
- net Pin_28: now also J5.13 (Pin_13), J6.13 (Pin_13)
- net Pin_29: now also J5.12 (Pin_12), J6.12 (Pin_12)
- net Pin_3: no longer J5.3 (Pin_3), J6.3 (Pin_3)
- net Pin_30: now also J5.11 (Pin_11), J6.11 (Pin_11)
- net Pin_31: now also J5.10 (Pin_10), J6.10 (Pin_10)
- net Pin_32: now also J5.9 (Pin_9), J6.9 (Pin_9)
- net Pin_33: now also J5.8 (Pin_8), J6.8 (Pin_8)
- net Pin_34: now also J5.7 (Pin_7), J6.7 (Pin_7)
- net Pin_35: now also J5.6 (Pin_6), J6.6 (Pin_6)
- net Pin_36: now also J5.5 (Pin_5), J6.5 (Pin_5)
- net Pin_37: now also J5.4 (Pin_4), J6.4 (Pin_4)
- net Pin_38: now also J5.3 (Pin_3), J6.3 (Pin_3)
- net Pin_39: now also J5.2 (Pin_2), J6.2 (Pin_2)
- net Pin_4: no longer J5.4 (Pin_4), J6.4 (Pin_4)
- net Pin_40: now also J5.1 (Pin_1), J6.1 (Pin_1)
- net Pin_5: no longer J5.5 (Pin_5), J6.5 (Pin_5)
- net Pin_6: no longer J5.6 (Pin_6), J6.6 (Pin_6)
- net Pin_7: no longer J5.7 (Pin_7), J6.7 (Pin_7)
- net Pin_8: no longer J5.8 (Pin_8), J6.8 (Pin_8)
- net Pin_9: no longer J5.9 (Pin_9), J6.9 (Pin_9)
- net VCC: now also D1.1 (K), JP1.2 (B)
- net VIN: now reaches J13.1 (Pin_1), J14.1, J15.1 (Pin_1), J16.1 (Pin_1)
- net VIN: now also SW1.2 (B)
- net IDC01 (R1) renamed IDC01
- net IDC02 (G1) renamed IDC02
- net IDC03 (B1) renamed IDC03
- net IDC05 (R2) renamed IDC05
- net IDC06 (G2) renamed IDC06
- net IDC07 (B2) renamed IDC07
- net IDC08 (E) renamed IDC08
- net IDC09 (A) renamed IDC09
- net IDC10 (B) renamed IDC10
- net IDC11 (C) renamed IDC11
- net IDC12 (D) renamed IDC12
- net IDC13 (CLK) renamed IDC13
- net IDC14 (LAT) renamed IDC14
- net IDC15 (OE) renamed IDC15
- now unconnected: J14.3
- no-connect marks 0 -> 3
Other:
- added sheet Lower IDC Pins Level Shifting (level_shifting.kicad_sch)
- added sheet Upper IDC Pins Level Shifting (level_shifting.kicad_sch)
- moved on the sheet: D1, J1, J2, J3, J4, J5, J6, J7, J8, JP1
