File: multi_expansion_board4/multi_expansion_board4.kicad_pcb (KiCad board)
At the start: 2 copper layers, 48.3 x 99.1 mm, 250 parts, among them J1 Conn_01x20, J10 Conn_01x20, J11 Conn_01x20, J12 Conn_01x20, J13 Conn_01x20, J14 Conn_01x20, J15 Conn_01x06, J16 Conn_01x06, J17 Conn_01x06, J18 Conn_01x06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

Commit message: Add .gitignore.
Parts:
- moved SW4 0.40 mm to (55.5, 156.1)
Routing:
- net Net-(D4-A): track 28.0 -> 27.2 mm
