File: ws8211_dumb_adaptor2/switch_unit.kicad_sch (KiCad schematic)
At the start: 14 parts, among them Q1 2TY, Q10 2N7002K, Q13 N-CHANNEL POWER MOSFET, Q19 2N7002K, Q3 2N7002K, Q7 2N7002K

Commit message: Add .gitignore.
Parts:
- renumbered Q7 to Q13, Q10 to Q14, Q13 to Q3, Q19 to Q7, Q3 to Q8
