File: ws8211_dumb_adaptor2/ws8211_dumb_adaptor2.kicad_pcb (KiCad board)
At the start: 2 copper layers, 48.3 x 48.3 mm, 66 parts, among them J1 Barrel_Jack_Switch, J2 Screw_Terminal_01x02, J3 Conn_01x03, J4 Conn_01x03, J5 Conn_01x04, J6 Conn_01x04, J7 Conn_01x02, J8 Conn_01x02, Q1 2TY, Q10 2N7002K, Q11 2N7002K, Q12 2N7002K, Q13 N-CHANNEL POWER MOSFET, Q14 N-CHANNEL POWER MOSFET, Q15 N-CHANNEL POWER MOSFET, Q19 2N7002K, Q2 2TY, Q20 2N7002K, Q21 2N7002K, Q3 2N7002K, Q4 2N7002K, Q5 2TY, Q6 2N7002K, Q7 2N7002K, Q8 2N7002K, Q9 2N7002K

Commit message: Add .gitignore.
Parts:
- moved J1 52.9 mm to (66.0, 64.8)
- moved J3 52.9 mm to (52.1, 73.7)
- moved J4 52.9 mm to (87.6, 73.7)
- moved J7 52.9 mm to (57.1, 102.9)
- moved Q15 52.9 mm to (71.8, 78.7)
- moved Q16 52.9 mm to (67.9, 78.7)
- moved Q17 52.9 mm to (61.6, 78.7)
- moved Q18 52.9 mm to (57.8, 78.7)
- moved R10 52.9 mm to (74.9, 90.8)
- moved R11 52.9 mm to (79.4, 90.8)
- moved R12 52.9 mm to (83.2, 90.8)
- moved R13 52.9 mm to (57.1, 90.8)
- moved R14 52.9 mm to (68.6, 90.8)
- moved R16 52.9 mm to (76.8, 90.8)
- moved R22 52.9 mm to (72.7, 83.8)
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- renumbered J5 to J1, J6 to J2, J7 to J5, J8 to J6, J2 to J7, J1 to J8, JP18 to JP1, JP19 to JP2, JP20 to JP3, JP21 to JP4, JP22 to JP5, Q15 to Q1, Q4 to Q10, Q21 to Q11, Q6 to Q12, Q7 to Q13, Q10 to Q14, Q8 to Q15, Q11 to Q16, Q9 to Q17, Q12 to Q18, Q14 to Q2, Q13 to Q3, Q2 to Q4, Q1 to Q5, Q5 to Q6, Q19 to Q7, Q3 to Q8, Q20 to Q9, R7 to R1, R3 to R10, R25 to R11, R22 to R12, R1 to R13, R4 to R14, R26 to R15, R23 to R16, R10 to R17, R5 to R18, R16 to R19, R8 to R2, R19 to R20, R13 to R21, R17 to R22, R11 to R23, R20 to R24, R14 to R25, R12 to R26, R18 to R27, R21 to R28, R15 to R29, R9 to R3, R29 to R4, R28 to R5, R2 to R7, R27 to R8, R24 to R9
Other:
- board text added: "POWER SELECT"
- board text added: "VEXT"
- board text added: "VINT"
- board text removed: "LOAD"
- board text removed: "VDD"
