File: ws8211_dumb_adaptor2/ws8211_dumb_adaptor2.kicad_sch (KiCad schematic)
At the start: 20 parts, among them J1 Barrel_Jack_Switch, J2 Screw_Terminal_01x02, J3 Conn_01x03, J4 Conn_01x03, J5 Conn_01x04, J6 Conn_01x04, J7 Conn_01x02, J8 Conn_01x02

Commit message: Add .gitignore.
Parts:
- renumbered J5 to J1, J6 to J2, J7 to J5, J8 to J6, J2 to J7, J1 to J8, JP18 to JP1, JP19 to JP2, JP20 to JP3, JP21 to JP4, JP22 to JP5, R7 to R1, R1 to R13, R8 to R2, R9 to R3, R2 to R7
Changed lines of the file:
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@@
   (symbol (lib_id "Connector_Generic:Conn_01x04") (at 278.13 104.14 0) (unit 1)
     (in_bom yes) (on_board yes) (dnp no) (fields_autoplaced)
-    (property "Reference" "J6" (at 280.67 106.045 0)
+    (property "Reference" "J2" (at 280.67 106.045 0)
       (effects (font (size 1.27 1.27)) (justify left))
     )
@@
       (project "ws8211_dumb_adaptor2"
         (path "/caeba6dc-40c7-4978-ae06-c328ef162ad3"
-          (reference "J6") (unit 1)
+          (reference "J2") (unit 1)
         )
       )
@@
   (symbol (lib_id "Jumper:SolderJumper_3_Open") (at 76.2 96.52 0) (unit 1)
     (in_bom yes) (on_board yes) (dnp no) (fields_autoplaced)
-    (property "Reference" "JP22" (at 76.2 91.44 0)
+    (property "Reference" "JP5" (at 76.2 91.44 0)
       (effects (font (size 1.27 1.27)))
     )
@@
       (project "ws8211_dumb_adaptor2"
         (path "/caeba6dc-40c7-4978-ae06-c328ef162ad3"
-          (reference "JP22") (unit 1)
+          (reference "JP5") (unit 1)
         )
       )
@@
   (symbol (lib_id "Connector_Generic:Conn_01x04") (at 269.24 104.14 0) (unit 1)
     (in_bom yes) (on_board yes) (dnp no) (fields_autoplaced)
-    (property "Reference" "J5" (at 271.78 106.045 0)
+    (property "Reference" "J1" (at 271.78 106.045 0)
       (effects (font (size 1.27 1.27)) (justify left))
     )
@@
       (project "ws8211_dumb_adaptor2"
         (path "/caeba6dc-40c7-4978-ae06-c328ef162ad3"
-          (reference "J5") (unit 1)
+          (reference "J1") (unit 1)
         )
       )
@@
   (symbol (lib_id "Jumper:SolderJumper_2_Bridged") (at 250.19 107.95 0) (unit 1)
     (in_bom yes) (on_board yes) (dnp no)
-    (property "Reference" "JP19" (at 250.19 105.41 0)
+    (property "Reference" "JP2" (at 250.19 105.41 0)
       (effects (font (size 1.27 1.27)))
     )
@@
       (project "ws8211_dumb_adaptor2"
         (path "/caeba6dc-40c7-4978-ae06-c328ef162ad3"
-          (reference "JP19") (unit 1)
+          (reference "JP2") (unit 1)
         )
       )
@@
   (symbol (lib_id "Device:R") (at 250.19 123.19 90) (unit 1)
     (in_bom yes) (on_board yes) (dnp no)
-    (property "Reference" "R9" (at 250.19 120.65 90)
+    (property "Reference" "R3" (at 250.19 120.65 90)
       (effects (font (size 1.27 1.27)))
     )
@@
       (project "ws8211_dumb_adaptor2"
         (path "/caeba6dc-40c7-4978-ae06-c328ef162ad3"
-          (reference "R9") (unit 1)
+          (reference "R3") (unit 1)
         )
       )
@@
   (symbol (lib_id "Device:R") (at 250.19 102.87 90) (unit 1)
     (in_bom yes) (on_board yes) (dnp no)
-    (property "Reference" "R7" (at 250.19 100.33 90)
+    (property "Reference" "R1" (at 250.19 100.33 90)
       (effects (font (size 1.27 1.27)))
     )
@@
       (project "ws8211_dumb_adaptor2"
         (path "/caeba6dc-40c7-4978-ae06-c328ef162ad3"
-          (reference "R7") (unit 1)
+          (reference "R1") (unit 1)
         )
       )
@@
   (symbol (lib_id "Jumper:SolderJumper_2_Bridged") (at 250.19 97.79 0) (unit 1)
     (in_bom yes) (on_board yes) (dnp no)
-    (property "Reference" "JP18" (at 250.19 95.25 0)
+    (property "Reference" "JP1" (at 250.19 95.25 0)
       (effects (font (size 1.27 1.27)))
     )
@@
       (project "ws8211_dumb_adaptor2"
         (path "/caeba6dc-40c7-4978-ae06-c328ef162ad3"
-          (reference "JP18") (unit 1)
+          (reference "JP1") (unit 1)
         )
       )
@@
   (symbol (lib_id "Jumper:Jumper_3_Open") (at 76.2 111.76 0) (unit 1)
     (in_bom yes) (on_board yes) (dnp no) (fields_autoplaced)
-    (property "Reference" "JP21" (at 76.2 106.68 0)
+    (property "Reference" "JP4" (at 76.2 106.68 0)
       (effects (font (size 1.27 1.27)))
     )
@@
       (project "ws8211_dumb_adaptor2"
         (path "/caeba6dc-40c7-4978-ae06-c328ef162ad3"
-          (reference "JP21") (unit 1)
+          (reference "JP4") (unit 1)
         )
       )
@@
   (symbol (lib_id "Connector_Generic:Conn_01x02") (at 21.59 120.65 0) (mirror y) (unit 1)
     (in_bom yes) (on_board yes) (dnp no)
-    (property "Reference" "J7" (at 21.59 128.27 0)
+    (property "Reference" "J5" (at 21.59 128.27 0)
       (effects (font (size 1.27 1.27)))
     )
@@
       (project "ws8211_dumb_adaptor2"
         (path "/caeba6dc-40c7-4978-ae06-c328ef162ad3"
-          (reference "J7") (unit 1)
+          (reference "J5") (unit 1)
         )
       )
@@
   (symbol (lib_id "Connector:Screw_Terminal_01x02") (at 21.59 96.52 0) (mirror y) (unit 1)
     (in_bom yes) (on_board yes) (dnp no)
-    (property "Reference" "J2" (at 22.86 93.98 0)
+    (property "Reference" "J7" (at 22.86 93.98 0)
       (effects (font (size 1.27 1.27)) (justify left))
     )
@@
       (project "ws8211_dumb_adaptor2"
         (path "/caeba6dc-40c7-4978-ae06-c328ef162ad3"
-          (reference "J2") (unit 1)
+          (reference "J7") (unit 1)
         )
       )
@@
   (symbol (lib_id "Jumper:SolderJumper_2_Bridged") (at 250.19 118.11 0) (unit 1)
     (in_bom yes) (on_board yes) (dnp no)
-    (property "Reference" "JP20" (at 250.19 115.57 0)
+    (property "Reference" "JP3" (at 250.19 115.57 0)
       (effects (font (size 1.27 1.27)))
     )
@@
       (project "ws8211_dumb_adaptor2"
         (path "/caeba6dc-40c7-4978-ae06-c328ef162ad3"
-          (reference "JP20") (unit 1)
+          (reference "JP3") (unit 1)
         )
       )
@@
   (symbol (lib_id "Device:R") (at 156.21 102.87 270) (mirror x) (unit 1)
     (in_bom yes) (on_board yes) (dnp no)
-    (property "Reference" "R2" (at 160.02 102.87 90)
+    (property "Reference" "R7" (at 160.02 102.87 90)
       (effects (font (size 1.27 1.27)))
     )
@@
       (project "ws8211_dumb_adaptor2"
         (path "/caeba6dc-40c7-4978-ae06-c328ef162ad3"
-          (reference "R2") (unit 1)
+          (reference "R7") (unit 1)
         )
       )
@@
   (symbol (lib_id "Connector:Barrel_Jack_Switch") (at 19.05 107.95 0) (unit 1)
     (in_bom yes) (on_board yes) (dnp no)
-    (property "Reference" "J1" (at 19.05 102.87 0)
+    (property "Reference" "J8" (at 19.05 102.87 0)
       (effects (font (size 1.27 1.27)))
     )
@@
       (project "ws8211_dumb_adaptor2"
         (path "/caeba6dc-40c7-4978-ae06-c328ef162ad3"
-          (reference "J1") (unit 1)
+          (reference "J8") (unit 1)
         )
       )
@@
   (symbol (lib_id "Device:R") (at 156.21 97.79 270) (mirror x) (unit 1)
     (in_bom yes) (on_board yes) (dnp no)
-    (property "Reference" "R1" (at 160.02 97.79 90)
+    (property "Reference" "R13" (at 160.02 97.79 90)
       (effects (font (size 1.27 1.27)))
     )
@@
       (project "ws8211_dumb_adaptor2"
         (path "/caeba6dc-40c7-4978-ae06-c328ef162ad3"
-          (reference "R1") (unit 1)
+          (reference "R13") (unit 1)
         )
       )
@@
   (symbol (lib_id "Connector_Generic:Conn_01x02") (at 40.64 120.65 0) (unit 1)
     (in_bom yes) (on_board yes) (dnp no) (fields_autoplaced)
-    (property "Reference" "J8" (at 43.18 121.285 0)
+    (property "Reference" "J6" (at 43.18 121.285 0)
       (effects (font (size 1.27 1.27)) (justify left))
     )
@@
       (project "ws8211_dumb_adaptor2"
         (path "/caeba6dc-40c7-4978-ae06-c328ef162ad3"
-          (reference "J8") (unit 1)
+          (reference "J6") (unit 1)
         )
       )
@@
   (symbol (lib_id "Device:R") (at 250.19 113.03 90) (unit 1)
     (in_bom yes) (on_board yes) (dnp no)
-    (property "Reference" "R8" (at 250.19 110.49 90)
+    (property "Reference" "R2" (at 250.19 110.49 90)
       (effects (font (size 1.27 1.27)))
     )
@@
       (project "ws8211_dumb_adaptor2"
         (path "/caeba6dc-40c7-4978-ae06-c328ef162ad3"
-          (reference "R8") (unit 1)
-        )
-      )
+          (reference "R2") (unit 1)
+        )
+      )
