File: level_shifter2/level_shifter2.kicad_pcb (KiCad board)
At the start: 2 copper layers, 15.2 x 17.8 mm, 8 parts, among them J1 Conn_01x04, J2 Conn_01x04, J3 Conn_01x06, Q1 BSS138

Commit message: Added bike light.
Other:
- board text removed: "JLCJLCJLCJLC"
Changed lines of the file:
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@@
     (effects (font (size 1 1) (thickness 0.15)) (justify bottom mirror))
-  )
-  (gr_text "JLCJLCJLCJLC" (at 109.22 76.2) (layer "B.SilkS")
-    (effects (font (size 0.8 0.8) (thickness 0.15)) (justify bottom mirror))
   )
   (gr_text "HS" (at 115.57 78.74) (layer "B.SilkS")
