File: slide_pot_breakout/slide_pot_breakout.kicad_pcb (KiCad board)
At the start: 2 copper layers, 73.7 x 24.1 mm, 10 parts, among them J1 Conn_01x03, J2 Conn_01x03, J3 Conn_01x03, J4 Conn_01x03, J6 Conn_01x06

Commit message: Added bike light.
Other:
- board text removed: "JLCJLCJLCJLC"
Changed lines of the file:
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@@
     (effects (font (size 1 1) (thickness 0.15)) (justify mirror))
-  )
-  (gr_text "JLCJLCJLCJLC" (at 78.74 73.66) (layer "B.SilkS")
-    (effects (font (size 0.8 0.8) (thickness 0.15)) (justify mirror))
   )
   (gr_text "2" (at 62.865 80.01 90) (layer "F.SilkS")
@@
     (pts (xy 41.91 83.82) (xy 41.91 59.69))
     (height -5.08)
-    (gr_text "24.1300 mm" (at 35.68 71.755 90) (layer "Cmts.User")
+    (gr_text "0.9500 in" (at 35.68 71.755 90) (layer "Cmts.User")
       (effects (font (size 1 1) (thickness 0.15)))
     )
@@
     (pts (xy 41.91 59.69) (xy 115.57 59.69))
     (height -5.08)
-    (gr_text "73.6600 mm" (at 78.74 53.46) (layer "Cmts.User")
+    (gr_text "2.9000 in" (at 78.74 53.46) (layer "Cmts.User")
       (effects (font (size 1 1) (thickness 0.15)))
     )
