File: bike_light/bike_light.kicad_pcb (KiCad board)
At the start: 2 copper layers, 96.5 x 30.5 mm, 31 parts, among them J1 USB_C_Receptacle_PowerOnly_6P, J2 USB_C_Receptacle_PowerOnly_6P, J3 Conn_01x02, J4 Conn_01x02, U1 LM317_TO-220, U2 LM317_TO-252

Commit message: Finish bike light.
Parts:
- J3, J4: footprint Connector_PinHeader_2.54mm:PinHeader_1x02_P2.54mm_Vertical -> Connector_Wire:SolderWire-0.75sqmm_1x02_P4.8mm_D1.25mm_OD2.3mm_Relief; moved to B.Cu
- moved C1 70.8 mm to (118.1, 68.6), turned to 0 degrees
- moved R8 18.5 mm to (42.5, 59.1), turned to 180 degrees
- moved R7 15.7 mm to (46.4, 59.1), turned to 180 degrees
- moved J4 14.6 mm to (118.1, 72.0), turned to -90 degrees
- moved J3 14.3 mm to (118.1, 60.3), turned to -90 degrees
- moved R6 7.85 mm to (42.5, 55.9), turned to 180 degrees
- moved R5 6.87 mm to (46.4, 55.9), turned to 180 degrees
- moved U1 4.58 mm to (41.9, 81.3)
- moved U2 4.58 mm to (44.5, 73.3)
Routing:
- net GND: track 300.0 -> 274.6 mm, vias 1 -> 0
- net +5V: track 148.7 -> 123.8 mm
- net SENSE: track 38.1 -> 26.6 mm
- net REG: track 227.0 -> 237.1 mm
Other:
- board size 96.5 x 30.5 mm -> 99.1 x 30.5 mm
- board text added: "+5V"
- board text added: "GND"
- board text added: "WayWayWay"
