File: bike_light/bike_light.kicad_sch (KiCad schematic)
At the start: 31 parts, among them J1 USB_C_Receptacle_PowerOnly_6P, J2 USB_C_Receptacle_PowerOnly_6P, J3 Conn_01x02, J4 Conn_01x02, U1 LM317_TO-220, U2 LM317_TO-252

Commit message: Finish bike light.
Parts:
- J3, J4: footprint Connector_PinHeader_2.54mm:PinHeader_1x02_P2.54mm_Vertical -> SolderWire-0.75sqmm_1x02_P4.8mm_D1.25mm_OD2.3mm_Relief
Changed lines of the file:
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@@
       (effects (font (size 1.27 1.27)) (justify left))
     )
-    (property "Footprint" "Connector_PinHeader_2.54mm:PinHeader_1x02_P2.54mm_Vertical" (at 163.83 81.28 0)
+    (property "Footprint" "SolderWire-0.75sqmm_1x02_P4.8mm_D1.25mm_OD2.3mm_Relief" (at 163.83 81.28 0)
       (effects (font (size 1.27 1.27)) hide)
     )
@@
       (effects (font (size 1.27 1.27)) (justify left))
     )
-    (property "Footprint" "Connector_PinHeader_2.54mm:PinHeader_1x02_P2.54mm_Vertical" (at 163.83 90.17 0)
-      (effects (font (size 1.27 1.27)) hide)
-    )
+    (property "Footprint" "SolderWire-0.75sqmm_1x02_P4.8mm_D1.25mm_OD2.3mm_Relief" (at 163.83 90.17 0)
+      (effects (font (size 1.27 1.27)) hide)
+    )
